Commit message: Imported upstream version '0.1.3' of 'upstream'

File: segbot_description/gazebo/common.gazebo.xacro (robot description, xacro)
@@ -2,5 +2,5 @@
 <root
   xmlns:xacro="http://ros.org/wiki/xacro">
-  <xacro:property name="SIMPLE_ROBOT_RADIUS" value="0.05" />
+  <xacro:property name="SIMPLE_ROBOT_RADIUS" value="0.30" />
   <xacro:macro name="gazebo_segbot_base_link_surface">
     <gazebo reference="base_link">
@@ -52,4 +52,7 @@
       <torque>20</torque>
       <commandTopic>cmd_vel</commandTopic>
+      <odometryTopic>odom</odometryTopic>
+      <odometryFrame>odom</odometryFrame>
+      <robotBaseFrame>base_footprint</robotBaseFrame>
     </plugin>
   </xacro:macro>
