Commit message: Imported upstream version '0.3.1' of 'upstream'

File: segbot_description/gazebo/segbot.gazebo.xacro (robot description, xacro)
@@ -57,7 +57,7 @@
     <xacro:unless value="$(arg use_full_gazebo_model)">
       <collision>
-        <origin xyz="0 0 0" rpy="0 0 0" />
-        <geometry>
-          <cylinder radius="0.305" length="0.4330" />
+        <origin xyz="0 0 -0.05" rpy="0 0 0" />
+        <geometry>
+          <cylinder radius="0.305" length="0.3330" />
         </geometry>
       </collision>
@@ -67,5 +67,5 @@
     <xacro:unless value="$(arg use_full_gazebo_model)">
       <joint name="laser_obstacle_joint" type="fixed">
-        <origin xyz="0.0 0 0.4165" rpy="0 0 0" />
+        <origin xyz="0.0 0 0.3165" rpy="0 0 0" />
         <parent link="base_link"/>
         <child link="laser_obstacle" />

File: segbot_description/robots/segbot_v2.urdf.xacro (robot description, xacro)
@@ -3,8 +3,8 @@
        xmlns:xacro="http://ros.org/wiki/xacro">
   <!-- Included URDF Files -->
-  <xacro:include filename="$(find segbot_description)/urdf/common.urdf.xacro" />
+  <xacro:include filename="$(find segbot_description)/urdf/v2/common.urdf.xacro" />
   <xacro:include filename="$(find segbot_description)/gazebo/segbot.gazebo.xacro" />
   <xacro:include filename="$(find segbot_description)/urdf/segbot_base.urdf.xacro" />
-  <xacro:include filename="$(find segbot_description)/urdf/segbot_chassis.urdf.xacro" />
+  <xacro:include filename="$(find segbot_description)/urdf/v2/segbot_chassis.urdf.xacro" />
   <xacro:include filename="$(find segbot_description)/urdf/mounts/hokuyo_mount.urdf.xacro" />
   <xacro:include filename="$(find segbot_description)/urdf/mounts/kinect_mount.urdf.xacro" />
@@ -16,10 +16,15 @@
   <!-- Add the forward facing kinect sensor for navigation -->
   <xacro:kinect_mount name="nav_kinect" parent="back_right_vertical_beam" length="${SENSOR_BEAM_LENGTH*INCH_TO_M}">
-    <origin xyz="0 ${0.5*INCH_TO_M} ${10.5*INCH_TO_M}" rpy="-${M_PI/2} -${M_PI/2} 0" />
+    <origin xyz="${1*INCH_TO_M} -${0.5*INCH_TO_M} ${11.5*INCH_TO_M}" rpy="-${M_PI/2} -${M_PI/2} 0" />
   </xacro:kinect_mount>
   <!-- Add the hokuyo -->
   <xacro:hokuyo_mount name="nav_hokuyo" parent="front_left_vertical_beam" length="${SENSOR_BEAM_LENGTH*INCH_TO_M}" ros_topic="scan" update_rate="10" min_angle="${-(5 * M_PI)/12}" max_angle="${(5 * M_PI)/12}">
-    <origin xyz="0 -${0.5*INCH_TO_M} ${7*INCH_TO_M}" rpy="${M_PI/2} ${M_PI/2} 0" />
+    <origin xyz="${1*INCH_TO_M} ${0.5*INCH_TO_M} ${4.5*INCH_TO_M}" rpy="${M_PI/2} ${M_PI/2} 0" />
   </xacro:hokuyo_mount>
+  <!-- Add a beam at top so that the robot looks complete. -->
+  <xacro:beam_8020 name="front_cap_beam" parent="front_right_vertical_beam" length="${SENSOR_BEAM_LENGTH*INCH_TO_M}">
+    <origin xyz="0 -${0.5*INCH_TO_M} ${36.5*INCH_TO_M}"
+      rpy="-${M_PI/2} 0 0" />
+  </xacro:beam_8020>
   <xacro:gazebo_segbot_ros_controllers />
 </robot>

Commit message: Imported upstream version '0.3.2' of 'upstream'

File: segbot_description/gazebo/segbot.gazebo.xacro (robot description, xacro)
@@ -42,5 +42,5 @@
         <inertia ixx="3000.0" ixy="0.0" ixz="0.0"
           iyy="3000.0" iyz="0.0"
-          izz="3000.0" />
+          izz="30.0" />
       </inertial>
     </xacro:unless>
@@ -174,10 +174,10 @@
     </xacro:if>
   </xacro:macro>
-  <xacro:macro name="standoff_632_collision" params="length">
+  <xacro:macro name="standoff_collision" params="radius length">
     <xacro:if value="$(arg use_full_gazebo_model)">
       <collision>
         <origin xyz="0 0 ${length/2}" rpy="0 0 0"/>
         <geometry>
-          <cylinder length="${length}" radius="0.003175" />
+          <cylinder length="${length}" radius="${radius}" />
         </geometry>
       </collision>
