Commit message: Imported upstream version '0.1.6' of 'upstream'

File: segbot_description/urdf/segbot_base.urdf.xacro (robot description, xacro)
@@ -3,5 +3,5 @@
       xmlns:xacro="http://ros.org/wiki/xacro">
   <!-- Included URDF Files -->
-  <include filename="$(find segbot_description)/urdf/segbot_wheel.urdf.xacro" />
+  <xacro:include filename="$(find segbot_description)/urdf/segbot_wheel.urdf.xacro" />
   <xacro:macro name="segbot">
     <!-- root link, on the ground just below the robot origin -->
@@ -21,11 +21,5 @@
     <!-- This is the robot origin, center of the 2 wheels (axis of rotation) -->
     <link name="base_link">
-      <inertial>
-        <mass value="30" />
-        <origin xyz="-0.1 0 -0.075" />
-        <inertia ixx="3.0" ixy="0.0" ixz="0.0"
-          iyy="3.0" iyz="0.0"
-          izz="2.0" />
-      </inertial>
+      <xacro:segbot_base_link_inertial />
       <visual>
         <origin xyz="0 0 0" rpy="0 0 0" />
