Commit message: Imported upstream version '0.2.0' of 'upstream'

File: segbot_description/robots/segbot_default.xacro (robot description, xacro)
@@ -1,3 +1,4 @@
 <?xml version="1.0"?>
+<!-- Standard (default) segbot configuration. -->
 <robot name="segbot"
        xmlns:xacro="http://ros.org/wiki/xacro">
@@ -7,5 +8,7 @@
   <xacro:include filename="$(find segbot_description)/urdf/segbot_base.urdf.xacro" />
   <xacro:include filename="$(find segbot_description)/urdf/segbot_chassis.urdf.xacro" />
+  <xacro:include filename="$(find segbot_description)/urdf/mounts/sensor_mount.urdf.xacro" />
   <xacro:include filename="$(find segbot_description)/urdf/mounts/hokuyo_mount.urdf.xacro" />
+  <xacro:include filename="$(find segbot_description)/urdf/mounts/kinect_mount.urdf.xacro" />
   <!-- Add the segbot base -->
   <xacro:segbot />
@@ -13,6 +16,15 @@
     <origin xyz="${BASE_PLATE_X_OFFSET*INCH_TO_M} 0 ${BASE_PLATE_Z_OFFSET*INCH_TO_M}"/>
   </xacro:segbot_chassis>
+  <xacro:sensor_mount name="sensor_mount" parent="chassis_mount_plate"/>
+  <!-- Add the forward facing kinect sensor for navigation -->
+  <xacro:kinect_mount name="nav_kinect" parent="back_right_vertical_beam"
+                      length="${SENSOR_BEAM_LENGTH*INCH_TO_M}">
+    <origin xyz="0 ${0.5*INCH_TO_M} ${10.5*INCH_TO_M}" rpy="-${M_PI/2} -${M_PI/2} 0" />
+  </xacro:kinect_mount>
   <!-- Add the hokuyo -->
-  <xacro:hokuyo_mount name="nav_hokuyo" parent="front_left_vertical_beam" length="${SENSOR_BEAM_LENGTH*INCH_TO_M}" ros_topic="scan" update_rate="10" min_angle="${-(5 * M_PI)/12}" max_angle="${(5 * M_PI)/12}">
+  <xacro:hokuyo_mount name="nav_hokuyo" parent="front_left_vertical_beam"
+                      length="${SENSOR_BEAM_LENGTH*INCH_TO_M}"
+                      ros_topic="scan" update_rate="10"
+                      min_angle="${-(5 * M_PI)/12}" max_angle="${(5 * M_PI)/12}">
     <origin xyz="0 -${0.5*INCH_TO_M} ${7*INCH_TO_M}" rpy="${M_PI/2} ${M_PI/2} 0" />
   </xacro:hokuyo_mount>
