Commit message: Rebase from 'release/indigo/segbot_description'

File: urdf/v2/segbot_chassis.urdf.arm.xacro (robot description, xacro)
@@ -73,5 +73,5 @@
     <!-- laptop -->
     <xacro:laptop name="laptop" parent="laptop_base_plate">
-      <origin xyz="-${2.1*INCH_TO_M} 0 ${0.125*INCH_TO_M}" rpy="0 0 0" />
+      <origin xyz="-${3.0*INCH_TO_M} 0 ${0.125*INCH_TO_M}" rpy="0 0 0" />
     </xacro:laptop>
   </xacro:macro>
